File: pcb/imu.kicad_sch (KiCad schematic)
At the start: 7 parts, among them U5 BNO08x

Commit message: [firmware/pcb] Initial firmware upload + fixed mistake in PCB + added errata documentation
Parts:
- R27: now not fitted
Changed lines of the file:
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@@
 		(in_bom yes)
 		(on_board yes)
-		(dnp no)
+		(dnp yes)
 		(property "Reference" "R27"
 			(at 71.12 74.9299 0)
